File: Buffer/Buffer - Rev D.kicad_pcb (KiCad board)
At the start: 4 copper layers, 40.9 x 15.5 mm, 85 parts, among them Q1 NFET_EPC2, Q2 NFET_EPC2, Q3 NFET_EPC2, Q4 NFET_EPC2, U1 Si8274, U2 Si8274

Commit message: updated pcb and test results and graphics
All relevant files up to charge injection journal
Parts:
- C0: renamed from 0.47uF1; value C -> 0.1uF
