File: Schematic and Layout/UnfolderBuffer.kicad_pcb (KiCad board)
At the start: 4 copper layers, 135 x 92 mm, 187 parts, among them J1 Conn_01x02, J2 Conn_01x02, J3 Conn_01x02, J4 HSEC8-160-1-L-DV-A-BL, J5 HSEC8-130-01-L-DV-A, Q1 NFET_GaNSystems, U1 TLV760 - 3.3V, U10 LM2937xMP, U11 ADuM5010, U12 Si8271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

Commit message: Data from lab
Uploading scope images from the data collected in lab
Parts:
- C58: value 1uF -> .01uF
- C59: value 1uF -> 0.1uF
- R30: value 150 -> 500
Changed lines of the file:
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@@
       (effects (font (size 0.6985 0.4445) (thickness 0.111125)))
     )
-    (fp_text value 1uF (at 0 1.5 180) (layer F.Fab)
+    (fp_text value .01uF (at 0 1.5 180) (layer F.Fab)
       (effects (font (size 1 1) (thickness 0.15)))
     )
@@
       (effects (font (size 0.6985 0.4445) (thickness 0.111125)))
     )
-    (fp_text value 1uF (at 0 1.5 90) (layer F.Fab)
+    (fp_text value 0.1uF (at 0 1.5 90) (layer F.Fab)
       (effects (font (size 1 1) (thickness 0.15)))
     )
@@
       (effects (font (size 0.6985 0.4445) (thickness 0.111125)))
     )
-    (fp_text value 150 (at 0 1.45 90) (layer F.Fab)
-      (effects (font (size 1 1) (thickness 0.15)))
-    )
+    (fp_text value 500 (at 0 1.45 90) (layer F.Fab)
+      (effects (font (size 1 1) (thickness 0.15)))
+    )

Commit message: updated pcb and test results and graphics
All relevant files up to charge injection journal
Parts:
- C57: value 1uF -> 0.1uF
