File: Schematic and Layout/UnfolderBuffer.sch (KiCad schematic (older format))
At the start: 34 parts, among them J1 Conn_01x02, J2 Conn_01x02, J3 Conn_01x02, U1 TLV760 - 3.3V

Commit message: updated pcb and test results and graphics
All relevant files up to charge injection journal
Parts:
- TP1, TP2, TP3, TP4: symbol user_tm:TP -> UnfolderBuffer-rescue:TP-user_tm
Changed lines of the file:
@@
 	2975 1875 2975 1925
 $Comp
-L user_tm:TP TP1
+L UnfolderBuffer-rescue:TP-user_tm TP1
 U 1 1 5C8C3760
 P 4100 1400
@@
 $EndComp
 $Comp
-L user_tm:TP TP2
+L UnfolderBuffer-rescue:TP-user_tm TP2
 U 1 1 5CE8E2CB
 P 4500 1725
@@
 Connection ~ 2825 2525
 $Comp
-L user_tm:TP TP3
+L UnfolderBuffer-rescue:TP-user_tm TP3
 U 1 1 5CEA191D
 P 3625 2275
@@
 $EndComp
 $Comp
-L user_tm:TP TP4
+L UnfolderBuffer-rescue:TP-user_tm TP4
 U 1 1 5CEA19B7
 P 3625 2525
